File: design/mosfets.sch (KiCad schematic (older format))
At the start: 15 parts, among them Q1 IRFS7530, Q2 IRFS7530, Q3 IRFS7530, Q4 IRFS7530, Q5 IRFS7530, Q6 IRFS7530

Commit message: Saved project with more recent version of KiCad. Added IRS2184 half bridge driver to BLDC_4_cache.lib
Parts:
- R28, R29, R30, R34, R35, R36, R42, R43, R46: symbol R -> R-RESCUE-BLDC_4
Changed lines of the file:
@@
 EESchema Schematic File Version 2
+LIBS:BLDC_4-rescue
 LIBS:power
 LIBS:device
@@
 LIBS:crf_1
 LIBS:BLDC_4-cache
-EELAYER 24 0
+EELAYER 25 0
 EELAYER END
 $Descr A4 11693 8268
@@
 $EndDescr
 $Comp
-L R R46
+L R-RESCUE-BLDC_4 R46
 U 1 1 53F8E60B
 P 7850 4050
@@
 $EndComp
 $Comp
-L R R30
+L R-RESCUE-BLDC_4 R30
 U 1 1 53F8E612
 P 4700 4050
@@
 $EndComp
 $Comp
-L R R29
+L R-RESCUE-BLDC_4 R29
 U 1 1 53F8E64B
 P 4400 3750
@@
 $EndComp
 $Comp
-L R R28
+L R-RESCUE-BLDC_4 R28
 U 1 1 53F8E652
 P 4400 2800
@@
 $EndComp
 $Comp
-L R R34
+L R-RESCUE-BLDC_4 R34
 U 1 1 53F8E65E
 P 5950 2800
@@
 $EndComp
 $Comp
-L R R35
+L R-RESCUE-BLDC_4 R35
 U 1 1 53F8E665
 P 5950 3750
@@
 $EndComp
 $Comp
-L R R43
+L R-RESCUE-BLDC_4 R43
 U 1 1 53F8E688
 P 7550 3750
@@
 $EndComp
 $Comp
-L R R42
+L R-RESCUE-BLDC_4 R42
 U 1 1 53F8E68F
 P 7550 2800
@@
 $EndComp
 $Comp
-L R R36
+L R-RESCUE-BLDC_4 R36
 U 1 1 53F8E69C
 P 5950 4050
@@
 00 00 00 41 83 58 05 00 00 08 1A C4 2A 00 00 40 D0 20 56 01 00 00 82 06 B1 0A 00 00 10 34 88 55
 00 00 80 A0 41 AC 02 00 00 04 CD FF 03 15 B2 0E 9E 1D 9F E2 F2 00 00 00 00 49 45 4E 44 AE 42 60
-82 FA
+82 5E
 EndData
 $EndBitmap
