File: design/BLDC_4.sch (KiCad schematic (older format))
At the start: 39 parts, among them K1 SERVO, P1 HALL, P10 CONN_1, P101 CANBUS, P11 CONN_1, P12 CONN_1, P13 CONN_1, P14 CONN_1, P15 CONN_1, P16 CONN_1, P17 CONN_1, P18 CONN_1, P3 PWR_COMM/USART1/Encoder, P4 IN+, P5 IN-, P6 MOTOR1, P7 MOTOR2, P8 Current sensors, P9 MOTOR3, X1 MINI-USB-SHIELD-32005-201

Commit message: Selected footprints
Parts:
- P10, P11, P12, P13, P14, P15, P16, P17, P18: value CONN_1 -> CONN_DRV; footprint (none) -> FootprintsBLDC:PAD_DRV
- P6: value MOTOR1 -> CONN_DRV
- P7: value MOTOR2 -> CONN_DRV
- P8: footprint (none) -> CRF1:MICRO_JST_6
- P9: value MOTOR3 -> CONN_DRV; footprint CRF1:1PAD_4x5mm -> FootprintsBLDC:PAD_DRV
- R103, R104, R37, R38: footprint SMD_Packages:SMD-0603_r -> Resistors_SMD:R_0603
- R14, R15, R16, R6: footprint (none) -> Resistors_SMD:R_0603
- R22, R3, R4, R5: footprint SMD_Packages:SMD-0603_r -> Resistors_SMD:R_0603_HandSoldering
Other:
- note added: "Goes to footprint"
- note added: "Not at footprint"
Changed lines of the file:
@@
 F 0 "R5" V 6500 5500 50  0000 C CNN
 F 1 "2k2" V 6600 5550 50  0000 C CNN
-F 2 "SMD_Packages:SMD-0603_r" H 6600 5550 60  0001 C CNN
+F 2 "Resistors_SMD:R_0603_HandSoldering" H 6600 5550 60  0001 C CNN
 F 3 "" H 6600 5550 60  0001 C CNN
 	1    6600 5550
@@
 F 0 "R4" V 2000 2050 50  0000 C CNN
 F 1 "2k2" V 2050 2250 50  0000 C CNN
-F 2 "SMD_Packages:SMD-0603_r" H 2050 2250 60  0001 C CNN
+F 2 "Resistors_SMD:R_0603_HandSoldering" H 2050 2250 60  0001 C CNN
 F 3 "" H 2050 2250 60  0001 C CNN
 	1    2050 2250
@@
 F 0 "R3" V 2000 1950 50  0000 C CNN
 F 1 "39k" V 2050 2150 50  0000 C CNN
-F 2 "SMD_Packages:SMD-0603_r" H 2050 2150 60  0001 C CNN
+F 2 "Resistors_SMD:R_0603_HandSoldering" H 2050 2150 60  0001 C CNN
 F 3 "" H 2050 2150 60  0001 C CNN
 	1    2050 2150
@@
 P 8450 2400
 F 0 "P9" H 8400 2450 40  0000 L CNN
-F 1 "MOTOR3" H 8450 2455 30  0001 C CNN
-F 2 "CRF1:1PAD_4x5mm" H 8450 2400 60  0001 C CNN
+F 1 "CONN_DRV" H 8450 2455 30  0001 C CNN
+F 2 "FootprintsBLDC:PAD_DRV" H 8450 2400 60  0001 C CNN
 F 3 "" H 8450 2400 60  0001 C CNN
 	1    8450 2400
@@
 P 8450 2150
 F 0 "P7" H 8400 2200 40  0000 L CNN
-F 1 "MOTOR2" H 8450 2205 30  0001 C CNN
+F 1 "CONN_DRV" H 8450 2205 30  0001 C CNN
 F 2 "CRF1:1PAD_4x5mm" H 8450 2150 60  0001 C CNN
 F 3 "" H 8450 2150 60  0001 C CNN
@@
 P 8450 1900
 F 0 "P6" H 8400 1950 40  0000 L CNN
-F 1 "MOTOR1" H 8450 1955 30  0001 C CNN
+F 1 "CONN_DRV" H 8450 1955 30  0001 C CNN
 F 2 "CRF1:1PAD_4x5mm" H 8450 1900 60  0001 C CNN
 F 3 "" H 8450 1900 60  0001 C CNN
@@
 F 0 "R103" V 2350 3250 40  0000 C CNN
 F 1 "22R" V 2407 3051 40  0000 C CNN
-F 2 "SMD_Packages:SMD-0603_r" V 2330 3050 30  0001 C CNN
+F 2 "Resistors_SMD:R_0603" V 2330 3050 30  0001 C CNN
 F 3 "" H 2400 3050 30  0000 C CNN
 	1    2400 3050
@@
 F 0 "R104" V 2350 3350 40  0000 C CNN
 F 1 "22R" V 2407 3151 40  0000 C CNN
-F 2 "SMD_Packages:SMD-0603_r" V 2330 3150 30  0001 C CNN
+F 2 "Resistors_SMD:R_0603" V 2330 3150 30  0001 C CNN
 F 3 "" H 2400 3150 30  0000 C CNN
 	1    2400 3150
@@
 F 0 "R38" V 5800 6400 50  0000 C CNN
 F 1 "100R" V 5900 6400 50  0000 C CNN
-F 2 "SMD_Packages:SMD-0603_r" H 5900 6400 60  0001 C CNN
+F 2 "Resistors_SMD:R_0603" H 5900 6400 60  0001 C CNN
 F 3 "" H 5900 6400 60  0001 C CNN
 	1    5900 6400
@@
 F 0 "R37" V 6100 6400 50  0000 C CNN
 F 1 "100R" V 6200 6400 50  0000 C CNN
-F 2 "SMD_Packages:SMD-0603_r" H 6200 6400 60  0001 C CNN
+F 2 "Resistors_SMD:R_0603" H 6200 6400 60  0001 C CNN
 F 3 "" H 6200 6400 60  0001 C CNN
 	1    6200 6400
@@
 F 0 "R22" V 6400 6400 50  0000 C CNN
 F 1 "2k2" V 6500 6400 50  0000 C CNN
-F 2 "SMD_Packages:SMD-0603_r" H 6500 6400 60  0001 C CNN
+F 2 "Resistors_SMD:R_0603_HandSoldering" H 6500 6400 60  0001 C CNN
 F 3 "" H 6500 6400 60  0001 C CNN
 	1    6500 6400
@@
 F 0 "R15" V 2930 5450 50  0000 C CNN
 F 1 "100" V 2850 5450 50  0000 C CNN
-F 2 "" V 2780 5450 30  0001 C CNN
+F 2 "Resistors_SMD:R_0603" V 2780 5450 30  0001 C CNN
 F 3 "" H 2850 5450 30  0000 C CNN
 	1    2850 5450
@@
 F 0 "R14" V 2580 5550 50  0000 C CNN
 F 1 "100" V 2500 5550 50  0000 C CNN
-F 2 "" V 2430 5550 30  0001 C CNN
+F 2 "Resistors_SMD:R_0603" V 2430 5550 30  0001 C CNN
 F 3 "" H 2500 5550 30  0000 C CNN
 	1    2500 5550
@@
 F 0 "P8" H 1100 6200 60  0000 C CNN
 F 1 "Current sensors" H 1100 6900 60  0000 C CNN
-F 2 "" H 1100 6550 60  0001 C CNN
+F 2 "CRF1:MICRO_JST_6" H 1100 6550 60  0001 C CNN
 F 3 "" H 1100 6550 60  0000 C CNN
 	1    1100 6550
@@
 F 0 "R16" V 2980 6400 50  0000 C CNN
 F 1 "100" V 2900 6400 50  0000 C CNN
-F 2 "" V 2830 6400 30  0001 C CNN
+F 2 "Resistors_SMD:R_0603" V 2830 6400 30  0001 C CNN
 F 3 "" H 2900 6400 30  0000 C CNN
 	1    2900 6400
@@
 F 0 "R6" V 1930 3350 50  0000 C CNN
 F 1 "10k" V 1850 3350 50  0000 C CNN
-F 2 "" V 1780 3350 30  0001 C CNN
+F 2 "Resistors_SMD:R_0603" V 1780 3350 30  0001 C CNN
 F 3 "" H 1850 3350 30  0000 C CNN
 	1    1850 3350
@@
 P 8450 2650
 F 0 "P10" H 8530 2650 40  0000 L CNN
-F 1 "CONN_1" H 8450 2705 30  0001 C CNN
-F 2 "" H 8450 2650 60  0001 C CNN
+F 1 "CONN_DRV" H 8450 2705 30  0001 C CNN
+F 2 "FootprintsBLDC:PAD_DRV" H 8450 2650 60  0001 C CNN
 F 3 "" H 8450 2650 60  0000 C CNN
 	1    8450 2650
@@
 P 8450 2950
 F 0 "P11" H 8530 2950 40  0000 L CNN
-F 1 "CONN_1" H 8450 3005 30  0001 C CNN
-F 2 "" H 8450 2950 60  0001 C CNN
+F 1 "CONN_DRV" H 8450 3005 30  0001 C CNN
+F 2 "FootprintsBLDC:PAD_DRV" H 8450 2950 60  0001 C CNN
 F 3 "" H 8450 2950 60  0000 C CNN
 	1    8450 2950
@@
 P 8450 3200
 F 0 "P12" H 8530 3200 40  0000 L CNN
-F 1 "CONN_1" H 8450 3255 30  0001 C CNN
-F 2 "" H 8450 3200 60  0001 C CNN
+F 1 "CONN_DRV" H 8450 3255 30  0001 C CNN
+F 2 "FootprintsBLDC:PAD_DRV" H 8450 3200 60  0001 C CNN
 F 3 "" H 8450 3200 60  0000 C CNN
 	1    8450 3200
@@
 P 8450 3450
 F 0 "P13" H 8530 3450 40  0000 L CNN
-F 1 "CONN_1" H 8450 3505 30  0001 C CNN
-F 2 "" H 8450 3450 60  0001 C CNN
+F 1 "CONN_DRV" H 8450 3505 30  0001 C CNN
+F 2 "FootprintsBLDC:PAD_DRV" H 8450 3450 60  0001 C CNN
 F 3 "" H 8450 3450 60  0000 C CNN
 	1    8450 3450
@@
 P 8450 3700
 F 0 "P14" H 8530 3700 40  0000 L CNN
-F 1 "CONN_1" H 8450 3755 30  0001 C CNN
-F 2 "" H 8450 3700 60  0001 C CNN
+F 1 "CONN_DRV" H 8450 3755 30  0001 C CNN
+F 2 "FootprintsBLDC:PAD_DRV" H 8450 3700 60  0001 C CNN
 F 3 "" H 8450 3700 60  0000 C CNN
 	1    8450 3700
@@
 P 8450 4000
 F 0 "P15" H 8530 4000 40  0000 L CNN
-F 1 "CONN_1" H 8450 4055 30  0001 C CNN
-F 2 "" H 8450 4000 60  0001 C CNN
+F 1 "CONN_DRV" H 8450 4055 30  0001 C CNN
+F 2 "FootprintsBLDC:PAD_DRV" H 8450 4000 60  0001 C CNN
 F 3 "" H 8450 4000 60  0000 C CNN
 	1    8450 4000
@@
 P 8450 4250
 F 0 "P16" H 8530 4250 40  0000 L CNN
-F 1 "CONN_1" H 8450 4305 30  0001 C CNN
-F 2 "" H 8450 4250 60  0001 C CNN
+F 1 "CONN_DRV" H 8450 4305 30  0001 C CNN
+F 2 "FootprintsBLDC:PAD_DRV" H 8450 4250 60  0001 C CNN
 F 3 "" H 8450 4250 60  0000 C CNN
 	1    8450 4250
@@
 P 8450 4500
 F 0 "P17" H 8530 4500 40  0000 L CNN
-F 1 "CONN_1" H 8450 4555 30  0001 C CNN
-F 2 "" H 8450 4500 60  0001 C CNN
+F 1 "CONN_DRV" H 8450 4555 30  0001 C CNN
+F 2 "FootprintsBLDC:PAD_DRV" H 8450 4500 60  0001 C CNN
 F 3 "" H 8450 4500 60  0000 C CNN
 	1    8450 4500
@@
 P 8450 4750
 F 0 "P18" H 8530 4750 40  0000 L CNN
-F 1 "CONN_1" H 8450 4805 30  0001 C CNN
-F 2 "" H 8450 4750 60  0001 C CNN
+F 1 "CONN_DRV" H 8450 4805 30  0001 C CNN
+F 2 "FootprintsBLDC:PAD_DRV" H 8450 4750 60  0001 C CNN
 F 3 "" H 8450 4750 60  0000 C CNN
 	1    8450 4750
@@
 Wire Wire Line
 	8300 4500 8000 4500
+Text Notes 1800 5250 0    60   ~ 0
+Not at footprint
+Text Notes 800  7050 0    60   ~ 0
+Goes to footprint
 $EndSCHEMATC
