File: design/temp.sch (KiCad schematic (older format))
At the start: 3 parts

Commit message: Saved project with more recent version of KiCad. Added IRS2184 half bridge driver to BLDC_4_cache.lib
Parts:
- C41: symbol C -> C-RESCUE-BLDC_4
- R1, R2: symbol R -> R-RESCUE-BLDC_4
Changed lines of the file:
@@
 EESchema Schematic File Version 2
+LIBS:BLDC_4-rescue
 LIBS:power
 LIBS:device
@@
 LIBS:crf_1
 LIBS:BLDC_4-cache
-EELAYER 24 0
+EELAYER 25 0
 EELAYER END
 $Descr A4 11693 8268
@@
 $EndDescr
 $Comp
-L R R1
+L R-RESCUE-BLDC_4 R1
 U 1 1 5426DA2F
 P 4400 3400
@@
 $EndComp
 $Comp
-L R R2
+L R-RESCUE-BLDC_4 R2
 U 1 1 5426DAA6
 P 4400 4100
@@
 $EndComp
 $Comp
-L C C41
+L C-RESCUE-BLDC_4 C41
 U 1 1 5426DADD
 P 4150 4100
@@
 $EndComp
 $Comp
-L GND #PWR024
+L GND-RESCUE-BLDC_4 #PWR024
 U 1 1 5426DB25
 P 4400 4600

Commit message: Assigned some footprints.
Parts:
- C41: footprint SMD_Packages:SMD-0603_c -> Capacitors_SMD:C_0603
Changed lines of the file:
@@
 F 0 "C41" H 4150 4200 40  0000 L CNN
 F 1 "2.2u" H 4156 4015 40  0000 L CNN
-F 2 "SMD_Packages:SMD-0603_c" H 4188 3950 30  0001 C CNN
+F 2 "Capacitors_SMD:C_0603" H 4188 3950 30  0001 C CNN
 F 3 "" H 4150 4100 60  0000 C CNN
 	1    4150 4100
@@
 $EndComp
 $Comp
-L VCC #PWR023
+L VCC #PWR020
 U 1 1 5426DB11
 P 4400 3050
-F 0 "#PWR023" H 4400 3150 30  0001 C CNN
+F 0 "#PWR020" H 4400 3150 30  0001 C CNN
 F 1 "VCC" H 4400 3150 30  0000 C CNN
 F 2 "" H 4400 3050 60  0000 C CNN
@@
 $EndComp
 $Comp
-L GND-RESCUE-BLDC_4 #PWR024
+L GND-RESCUE-BLDC_4 #PWR021
 U 1 1 5426DB25
 P 4400 4600
-F 0 "#PWR024" H 4400 4600 30  0001 C CNN
+F 0 "#PWR021" H 4400 4600 30  0001 C CNN
 F 1 "GND" H 4400 4530 30  0001 C CNN
 F 2 "" H 4400 4600 60  0000 C CNN

Commit message: Selected footprints
Parts:
- R1, R2: footprint SMD_Packages:SMD-0603_r -> Resistors_SMD:R_0603_HandSoldering
Changed lines of the file:
@@
 F 0 "R1" V 4480 3400 40  0000 C CNN
 F 1 "NTC 10k" V 4407 3401 40  0000 C CNN
-F 2 "SMD_Packages:SMD-0603_r" V 4330 3400 30  0001 C CNN
+F 2 "Resistors_SMD:R_0603_HandSoldering" V 4330 3400 30  0001 C CNN
 F 3 "" H 4400 3400 30  0000 C CNN
 	1    4400 3400
@@
 F 0 "R2" V 4480 4100 40  0000 C CNN
 F 1 "10k" V 4407 4101 40  0000 C CNN
-F 2 "SMD_Packages:SMD-0603_r" V 4330 4100 30  0001 C CNN
+F 2 "Resistors_SMD:R_0603_HandSoldering" V 4330 4100 30  0001 C CNN
 F 3 "" H 4400 4100 30  0000 C CNN
 	1    4400 4100
